File: pcb/pcb.kicad_pcb (KiCad board)
At the start: 4 copper layers, 100 x 50 mm, 71 parts, among them J1 DC 7-30V, J2 AC current input, J3 UART, J5 USB JTAG/Serial, SW1 RESET, SW2 BOOT, U1 ESP32-S3-WROOM-1, U2 USBLC6-2SC6, U3 AMS1117-3.3, U4 AP63205WU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

Commit message: PCB updated:
Revision 1.1
- Corrected footprint of the LC Tech HW-697 module
- Moved HW-697 signal output track to the In2.Cu layer

Previous updates:
- Justified length of the USB D+/D- tracks
Parts:
- U6: value LC_Tech_ZMPT101B_LM358_Sensor -> LC_Tech_HW697_Module; footprint footprints:LC_Tech_ZMPT101B_LM358_Sensor -> footprints:LC_Tech_HW697_Module
Routing:
- net AC_I: track 61.4 -> 67.4 mm
- net AC_V: track 56.1 -> 50.4 mm
- net +5VA: track 25.2 -> 23.7 mm
- net Net-(U6-OUT): track 19.0 -> 19.7 mm, vias 0 -> 1
Other:
- board text added: "${TITLE} Board Rev. ${REVISION}"
- board text added: "HW-697 Transformer Module"
- board text removed: "LC Tech ZMPT101B/LM358"
- board text removed: "Transformer Module"
